File: KiCad/Project2.1.sch (KiCad schematic (older format))
At the start: 91 parts, among them IC1 LT1308, IC2 TP4056, IC3 DW01A-G, J2 282836-9, J3 Gas Sensor, J4 Digital, J5 SIM, J6 Conn_Coaxial, J7 USB, J8 Power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

Commit message: Adding Principle of operation
Parts:
- C1: value 100uF Tantal ESR -> 470uF Tantal ESR
- C12: value 47uF -> 470uF
- D10: value NET -> CHRG
- D12: value STATUS -> Modem Status
- D8: value Status LED -> System Status
- D9: value STATUS -> PWR
- IC1: symbol LT1308ACS8#PBF:LT1308ACS8#PBF -> Project2.0-rescue:LT1308ACS8#PBF-LT1308ACS8#PBF
- J9: value Power -> Power 5V DC
- R25: value 1k -> 1.2k
Connections:
- wire segments 435 -> 436
- no-connect marks 101 -> 100
Changed lines of the file:
@@
 EESchema Schematic File Version 4
-LIBS:Project1.11-cache
+LIBS:Project2.1-cache
 EELAYER 30 0
 EELAYER END
@@
 Title "Gas Warning System board"
 Date "2019-10-08"
-Rev "1.0"
+Rev "2.1"
 Comp ""
 Comment1 ""
@@
 P 8200 1000
 F 0 "C1" H 8250 1100 50  0000 L CNN
-F 1 "100uF Tantal ESR" H 8100 700 50  0000 L CNN
+F 1 "470uF Tantal ESR" H 8100 700 50  0000 L CNN
 F 2 "Capacitor_Tantalum_SMD:CP_EIA-7343-31_Kemet-D" H 8238 850 50  0001 C CNN
 F 3 " T494C107K010AT" H 8200 1000 50  0001 C CNN
@@
 $EndComp
 Wire Wire Line
-	9800 2250 9650 2250
-Wire Wire Line
 	9200 2250 9150 2250
 Wire Wire Line
@@
 Wire Wire Line
 	9200 2350 8950 2350
-Wire Wire Line
-	9800 2650 9500 2650
 Wire Wire Line
 	9200 2650 8750 2650
@@
 Wire Wire Line
 	9550 2050 9550 2350
-Connection ~ 9550 2350
 Wire Wire Line
 	9550 2350 9500 2350
@@
 L power:Earth #PWR09
 U 1 1 5DA79346
-P 9650 2500
-F 0 "#PWR09" H 9650 2250 50  0001 C CNN
-F 1 "Earth" H 9650 2350 50  0001 C CNN
-F 2 "" H 9650 2500 50  0001 C CNN
-F 3 "~" H 9650 2500 50  0001 C CNN
-	1    9650 2500
-	1    0    0    -1
-$EndComp
-Wire Wire Line
-	9650 2450 9650 2500
+P 10950 1650
+F 0 "#PWR09" H 10950 1400 50  0001 C CNN
+F 1 "Earth" H 10950 1500 50  0001 C CNN
+F 2 "" H 10950 1650 50  0001 C CNN
+F 3 "~" H 10950 1650 50  0001 C CNN
+	1    10950 1650
+	1    0    0    -1
+$EndComp
 $Comp
 L Device:C C6
@@
 P 9450 3500
 F 0 "D12" H 9450 3400 50  0000 C CNN
-F 1 "STATUS" H 9100 3400 50  0000 C CNN
+F 1 "Modem Status" H 9100 3400 50  0000 C CNN
 F 2 "Diode_SMD:D_1206_3216Metric" H 9450 3500 50  0001 C CNN
 F 3 "~" H 9450 3500 50  0001 C CNN
@@
 P 6600 5100
 F 0 "D9" H 6600 5000 50  0000 C CNN
-F 1 "STATUS" V 6600 5350 50  0000 C CNN
+F 1 "PWR" V 6600 5350 50  0000 C CNN
 F 2 "Diode_SMD:D_1206_3216Metric" H 6600 5100 50  0001 C CNN
 F 3 "~" H 6600 5100 50  0001 C CNN
@@
 P 6800 5100
 F 0 "D10" H 6800 5000 50  0000 C CNN
-F 1 "NET" V 6800 4850 50  0000 C CNN
+F 1 "CHRG" V 6800 4850 50  0000 C CNN
 F 2 "Diode_SMD:D_1206_3216Metric" H 6800 5100 50  0001 C CNN
 F 3 "~" H 6800 5100 50  0001 C CNN
@@
 P 8300 5500
 F 0 "R25" V 8200 5400 50  0000 C CNN
-F 1 "1k" V 8200 5600 50  0000 C CNN
+F 1 "1.2k" V 8200 5600 50  0000 C CNN
 F 2 "Resistor_SMD:R_1206_3216Metric" V 8230 5500 50  0001 C CNN
 F 3 "~" H 8300 5500 50  0001 C CNN
@@
 Connection ~ 8700 5550
 $Comp
-L LT1308ACS8#PBF:LT1308ACS8#PBF IC1
+L Project2.0-rescue:LT1308ACS8#PBF-LT1308ACS8#PBF IC1
 U 1 1 5DB97CBA
 P 2350 1450
@@
 	1250 1250 1050 1250
 Wire Wire Line
-	1050 750  1050 1250
+	1050 750  1050 950
 Wire Wire Line
 	2350 1350 2700 1350
@@
 U 1 1 5DD6DEF9
 P 1050 1500
-F 0 "C12" H 1168 1546 50  0000 L CNN
-F 1 "47uF" H 1168 1455 50  0000 L CNN
+F 0 "C12" H 1200 1450 50  0000 L CNN
+F 1 "470uF" H 1150 1350 50  0000 L CNN
 F 2 "Capacitor_Tantalum_SMD:CP_EIA-7343-31_Kemet-D" H 1088 1350 50  0001 C CNN
 F 3 "~" H 1050 1500 50  0001 C CNN
@@
 P 6050 4000
 F 0 "D8" V 6050 3900 50  0000 C CNN
-F 1 "Status LED" V 6150 3800 50  0000 C CNN
+F 1 "System Status" V 6150 3800 50  0000 C CNN
 F 2 "Diode_SMD:D_1206_3216Metric" H 6050 4000 50  0001 C CNN
 F 3 "~" H 6050 4000 50  0001 C CNN
@@
 NoConn ~ 4950 4200
 NoConn ~ 4950 4300
-NoConn ~ 2350 1250
 NoConn ~ 1250 1350
 NoConn ~ 1250 1450
@@
 Wire Wire Line
 	8450 5850 8450 5200
-$Comp
-L 47553-1001:47553-1001 J5
-U 1 1 5DF493F0
-P 9950 2150
-F 0 "J5" H 10700 2450 50  0000 C CNN
-F 1 "SIM" H 10750 2350 50  0000 C CNN
-F 2 "47553-1001:475531001" H 10900 2250 50  0001 L CNN
-F 3 "https://componentsearchengine.com/Datasheets/1/47553-1001.pdf" H 10900 2150 50  0001 L CNN
-F 4 "1.27mm Pitch SIM Card Holder Push-Push" H 10900 2050 50  0001 L CNN "Description"
-F 5 "1" H 10900 1950 50  0001 L CNN "Height"
-F 6 "538-47553-1001" H 10900 1850 50  0001 L CNN "Mouser Part Number"
-F 7 "https://www.mouser.com/Search/Refine.aspx?Keyword=538-47553-1001" H 10900 1750 50  0001 L CNN "Mouser Price/Stock"
-F 8 "Molex" H 10900 1650 50  0001 L CNN "Manufacturer_Name"
-F 9 "47553-1001" H 10900 1550 50  0001 L CNN "Manufacturer_Part_Number"
-	1    9950 2150
-	1    0    0    -1
-$EndComp
 Wire Wire Line
 	11050 2650 11050 2800
@@
 L power:Earth #PWR051
 U 1 1 5DFFE6E5
-P 10500 2850
-F 0 "#PWR051" H 10500 2600 50  0001 C CNN
-F 1 "Earth" H 10500 2700 50  0001 C CNN
-F 2 "" H 10500 2850 50  0001 C CNN
-F 3 "~" H 10500 2850 50  0001 C CNN
-	1    10500 2850
-	1    0    0    -1
-$EndComp
-Wire Wire Line
-	10500 2850 10500 2800
+P 10500 2950
+F 0 "#PWR051" H 10500 2700 50  0001 C CNN
+F 1 "Earth" H 10500 2800 50  0001 C CNN
+F 2 "" H 10500 2950 50  0001 C CNN
+F 3 "~" H 10500 2950 50  0001 C CNN
+	1    10500 2950
+	1    0    0    -1
+$EndComp
 Connection ~ 10500 2800
 Wire Wire Line
@@
 Wire Wire Line
 	9750 2150 9950 2150
-Wire Wire Line
-	11050 2150 11050 2000
-Wire Wire Line
-	11050 2000 9800 2000
-Wire Wire Line
-	9800 2000 9800 2250
-Wire Wire Line
-	9950 2250 9850 2250
-Wire Wire Line
-	9850 2250 9850 2350
-Wire Wire Line
-	9550 2350 9850 2350
-Wire Wire Line
-	9950 2350 9900 2350
-Wire Wire Line
-	9900 2350 9900 2450
-Wire Wire Line
-	9650 2450 9900 2450
-Wire Wire Line
-	9950 2450 9950 2500
-Wire Wire Line
-	9950 2500 9800 2500
-Wire Wire Line
-	9800 2500 9800 2650
 NoConn ~ 11050 2250
-NoConn ~ 11050 2350
+NoConn ~ 9950 2450
 NoConn ~ 11050 2450
 NoConn ~ 11050 2550
@@
 P 10500 950
 F 0 "J9" H 10850 1200 50  0000 L CNN
-F 1 "Power" H 10800 1100 50  0000 L CNN
+F 1 "Power 5V DC" H 10800 1100 50  0000 L CNN
 F 2 "CON-SOCJ-2155:CONSOCJ2155" H 11150 800 50  0001 L CNN
 F 3 "http://www.produktinfo.conrad.com/datenblaetter/1500000-1599999/001582350-da-01-en-DC_EINBAUBUCHSE__SCHALTER_GESCHLOSSEN.pdf" H 11150 700 50  0001 L CNN
@@
 Wire Wire Line
 	5000 7000 5950 7000
+Wire Wire Line
+	2350 1250 2400 1250
+Wire Wire Line
+	2400 1250 2400 950
+Wire Wire Line
+	2400 950  1050 950
+Connection ~ 1050 950
+Wire Wire Line
+	1050 950  1050 1250
+$Comp
+L 47553-1001:47553-1001 J5
+U 1 1 5DF493F0
+P 9950 2150
+F 0 "J5" H 10700 2450 50  0000 C CNN
+F 1 "SIM" H 10750 2350 50  0000 C CNN
+F 2 "47553-1001:475531001" H 10900 2250 50  0001 L CNN
+F 3 "https://componentsearchengine.com/Datasheets/1/47553-1001.pdf" H 10900 2150 50  0001 L CNN
+F 4 "1.27mm Pitch SIM Card Holder Push-Push" H 10900 2050 50  0001 L CNN "Description"
+F 5 "1" H 10900 1950 50  0001 L CNN "Height"
+F 6 "538-47553-1001" H 10900 1850 50  0001 L CNN "Mouser Part Number"
+F 7 "https://www.mouser.com/Search/Refine.aspx?Keyword=538-47553-1001" H 10900 1750 50  0001 L CNN "Mouser Price/Stock"
+F 8 "Molex" H 10900 1650 50  0001 L CNN "Manufacturer_Name"
+F 9 "47553-1001" H 10900 1550 50  0001 L CNN "Manufacturer_Part_Number"
+	1    9950 2150
+	1    0    0    -1
+$EndComp
+Wire Wire Line
+	11050 2150 11100 2150
+Wire Wire Line
+	11100 2150 11100 1600
+Wire Wire Line
+	11100 1600 10950 1600
+Wire Wire Line
+	10950 1600 10950 1650
+Wire Wire Line
+	9650 2250 9950 2250
+Wire Wire Line
+	9950 2350 9550 2350
+Connection ~ 9550 2350
+Wire Wire Line
+	11050 2350 11100 2350
+Wire Wire Line
+	11100 2350 11100 2850
+Wire Wire Line
+	11100 2850 10500 2850
+Wire Wire Line
+	9850 2850 9850 2650
+Wire Wire Line
+	9500 2650 9850 2650
+Wire Wire Line
+	10500 2850 9850 2850
+Wire Wire Line
+	10500 2800 10500 2950
 $EndSCHEMATC
